File: ergo_60_case.kicad_pcb (KiCad board)
At the start: 2 copper layers, 285 x 94.6 mm, 166 parts, among them SW1 SW_Push, U1 PRTR5V0U2X, U2 OLED_SSD1306, U3 AT90USB1286-AU, U4 AVR-ISP, Y1 16MHz

Commit message: updating footprints for proper clearance
Parts:
- U3: footprint KiCadLibs:AT90USB1286-AU_QFP80P1600X1600X120-64N -> KiCadLibs:AT90USB1286-AU_TQFP_16X16-64N
- USB1: footprint Type-C:HRO-TYPE-C-31-M-12-Assembly -> KiCadLibs:HRO-TYPE-C-31-M-12_.25clearance
